Commit message: robot movement

File: robot_gazebo/urdf/robot.urdf.xacro (robot description, xacro)
@@ -153,4 +153,12 @@
         <cylinder radius="0.1" length="0.05"/>
       </geometry>
+      <surface>
+        <friction>
+          <ode>
+            <mu>1.0</mu>
+            <mu2>1.0</mu2>
+          </ode>
+        </friction>
+      </surface>
     </collision>
     <inertial>
@@ -173,4 +181,12 @@
         <cylinder radius="0.1" length="0.05"/>
       </geometry>
+      <surface>
+        <friction>
+          <ode>
+            <mu>1.0</mu>
+            <mu2>1.0</mu2>
+          </ode>
+        </friction>
+      </surface>
     </collision>
     <inertial>
@@ -196,7 +212,5 @@
   <gazebo>
     <plugin name="differential_drive_controller" filename="libgazebo_ros_diff_drive.so">
-      <ros>
-        <namespace>/</namespace>
-      </ros>
+      <update_rate>30</update_rate>
       <left_joint>left_wheel_joint</left_joint>
       <right_joint>right_wheel_joint</right_joint>
@@ -214,7 +228,3 @@
     </plugin>
   </gazebo>
-  <!-- Gazebo Material -->
-  <gazebo>
-    <material>Gazebo/Blue</material>
-  </gazebo>
 </robot>
